File: HW/BP_MCU.brd (EAGLE design)
At the start: 99.5 x 50.6 mm, 45 parts, among them Q1 8MHz, Q2 2N7002, Q3 2N7002, U1 STM32F103C8T6LQFP48_STM, U2 1-1825910-0

Commit message: Verze zadaná do výroby
Parts:
- added R12, R13: (no value), rcl:R0805
- added U$6: USBLC6-2, ESD:SOT23-6L
- C13, C15: value 4u7 -> 2u2
- moved C6 2.57 mm to (24.4, 37.5), turned to 180 degrees
- moved L1 0.38 mm to (10.2, 26.4)
- moved C12 0.38 mm to (11.4, 30.7)
Connections:
- new net DATA_N_U: U$1.A7, U$1.B7, U$6.1
- new net DATA_P_U: U$1.A6, U$1.B6, U$6.3
- new net N$5: C12.2, R12.2
- new net N$7: C17.2, R13.2
- net DATA_N: now also U$6.6; no longer U$1.A7, U$1.B7
- net DATA_P: now also U$6.4; no longer U$1.A6, U$1.B6
- net GND: now also R12.1, R13.1, U$6.2; no longer C12.2, C17.2
- net VBUS: now also U$6.5
Routing:
- net DATA_P: track 30.3 -> 15.2 mm
- net DATA_N: track 24.8 -> 10.2 mm
- net DATA_P_U: track 0.00 -> 12.5 mm
- net DATA_N_U: track 0.00 -> 12.5 mm
- net VBUS: track 13.2 -> 25.2 mm
- net N$5: track 0.00 -> 2.38 mm
- net N$7: track 0.00 -> 2.25 mm
- net +3V3: track 246.5 -> 245.3 mm
- net +5V: track 100.6 -> 101.6 mm
- net GND: track 65.2 -> 65.8 mm, vias 22 -> 23
