File: HW/snimaci_cast.sch (EAGLE design)
At the start: 76 parts, among them K1 G5LE, K2 G5LE, Q1 2N7002, Q3 2N7002

Commit message: Přidáno propojení desek fastony a distančními sloupky, změněna logika vyhodnocení nežádoucích stavů
Parts:
- removed PAD3, PAD4, PAD7, PAD8: (no value), wirepad:2,15/1,0
- removed U$3: SN74LVC2GU04, TI_logic:SN74LVC2GU04
- added C14, C15: u1, rcl:C-EUC0805
- added IC1, IC2: 7402D, 74xx-eu:7402D
- added X1, X2: (no value), con-rib:SH5-2
Connections:
- new net N$24: IC1A.I1, IC1B.O
- new net N$26: IC1C.O, IC1D.I0
- new net Q_1: IC1A.O, IC1B.I0, IC2D.I0
- new net Q_2: IC1C.I1, IC1D.O, IC2C.I0
- new net ZKRATOVANI_1: IC2A.O, Q3.G
- new net ZKRATOVANI_2: IC2B.O, Q1.G
- net +3V3: now also C14.1, C15.1, IC1P.VCC, IC2P.VCC; no longer U$3G$3.VCC
- net A1_IN: now also X1-1.1, X1-1.2; no longer PAD3.P
- net A2_IN: now also X2-1.1, X2-1.2; no longer PAD7.P
- net AGND: now also X1-2.1, X1-2.2, X2-2.1, X2-2.2; no longer PAD4.P, PAD8.P
- net EN1: now also IC2A.I0, IC2A.I1, IC2D.O; no longer U$3G$1.O
- net EN2: now also IC2B.I0, IC2B.I1, IC2C.O; no longer U$3G$2.O
- net GND: now also C14.2, C15.2, IC1P.GND, IC2P.GND; no longer U$3G$3.GND
- net INT1: now also IC1B.I1
- net INT2: now also IC1C.I0
- net PROT1: now also IC1A.I0, IC2D.I1; no longer Q3.G, U$3G$1.I
- net PROT2: now also IC1D.I1, IC2C.I1; no longer Q1.G, U$3G$2.I
Other:
- note added: "1.1"
- note added: "29.10.2024"
- note added: "Logika vyhodnocení přetečení prodového rozsahu"
- note added: "RS"
- note added: "Snímací část"
- note added: "Zkratování Bočníku"
- note removed: "DC-DC"
- note removed: "Napájení OZ"
- note removed: "Negace PROT pro vypnutí OZ"
- note removed: "Snímání vstupního výkonu"
- note removed: "Zkratování bočníku"
- moved on the sheet: C1, C10, C11, C12, C13, C2, C3, C4, C5, C6, C7, C8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

Commit message: Verze zadaná do výroby
Parts:
- added R35: (no value), rcl:R-EU_R0805
- C1, C11, C14, C15: value u1 -> 100n
- C10, C2, C3, C4, C5, C6, C7, C8, C9: value (none) -> 100n
- R10, R16, R2, R5: value (none) -> 1K
- R11, R12, R6, R8: value (none) -> 550R
- R13: value (none) -> 15K
- R14: value (none) -> 820R
- R15: value (none) -> 500R
- R17, R18: value (none) -> 5K
Connections:
- net AGND: now also R35.1
- net GND: now also R35.2
Other:
- moved on the sheet: JP1, JP3
