File: HW/BP_MCU.sch (EAGLE design)
At the start: 41 parts, among them Q1 8MHz, Q2 2N7002, Q3 2N7002, U1 STM32F103C8T6LQFP48_STM, U2 1-1825910-0

Commit message: Vytvoření ovládací desky, simulace a úprava filtrů
Parts:
- added C17: 4u7, rcl:C-EUC0805
- added JP4: (no value), pinhead:PINHD-2X4
- added L2: 47u, Induktory:AMRM00101040470MA1
- added R11: 0R, rcl:R-EU_R0805
- C11: device rcl:C-EUC0805 -> resistor:C-EUC0805
- C12: device rcl:CPOL-EUUD-8X10 -> resistor:C-EUC0805
- C13, C15: value 1u -> 4u7; device rcl:CPOL-EUUD-8X10 -> rcl:C-EUC0805
- C14, C16: value 1u -> 470n; device rcl:CPOL-EUUD-8X10 -> rcl:C-EUC0805
- JP2: device pinhead:PINHD-2X5/90 -> pinhead:PINHD-2X5
Connections:
- new net N$6: C11.1, C12.1, L1.2, L2.1, R11.1
- new net RIZENI_IN: JP4.5, U1A.PA4
- new net RIZENI_OUT: JP4.4, U1A.PA6
- new net STAV_IN: JP4.3, U1A.PA3
- new net STAV_OUT: JP4.6, U1A.PA5
- net +3V3: now also C13.1, JP4.7; no longer C13.+
- net +5V: now also C14.1, C16.1, C17.1, JP4.1, L2.2, R11.2; no longer C11.1, C12.+, C14.+, C16.+, L1.2
- net A3V3: now also C15.1; no longer C15.+
- net BOOT0: now also R1.2, S1.2; no longer R2.2, S1.1
- net BOOT1: now also R2.2, S1.1; no longer R1.2, S1.2
- net GND: now also C12.2, C13.2, C14.2, C15.2, C16.2, C17.2, JP4.2, JP4.8; no longer C12.-, C13.-, C14.-, C15.-, C16.-
- net PROT1: now also U1A.PB12; no longer U1A.PB13
- net PROT2: now also U1A.PB14; no longer U1A.PB15
- net RELE1_SIG: now also U1A.PB13; no longer U1A.PB12
- net RELE2_SIG: now also U1A.PB15; no longer U1A.PB14
Other:
- note added: "Konektor ochran"
- note added: "alternativně TLV76133DCYR"
- note removed: "Důraz na PSRR"

Commit message: Verze zadaná do výroby
Parts:
- added R12, R13: (no value), rcl:R-EU_R0805
- added U$6: USBLC6-2, ESD:USBLC6-2
- C13, C15: value 4u7 -> 2u2
Connections:
- new net DATA_N_U: U$1.D-, U$6.I1
- new net DATA_P_U: U$1.D+, U$6.I2
- new net N$5: C12.2, R12.2
- new net N$7: C17.2, R13.2
- net DATA_N: now also U$6.O1; no longer U$1.D-
- net DATA_P: now also U$6.O2; no longer U$1.D+
- net GND: now also R12.1, R13.1, U$6.GND; no longer C12.2, C17.2
- net VBUS: now also U$6.5V
Other:
- note added: "Vstupní filtr"
- note removed: "PÍ-článek"
- moved on the sheet: C10, C11, C12, C17, L1, L2, R11

Commit message: Přidání kostry FW v modifikaci pro provoz v konzoli
Other:
- note added: "2.1.2025"
- note added: "MCU a napájení"
- note added: "V případě osazení L2 je R11 ponechán neosazený"
- moved on the sheet: C10, C11, C12, C13, C14, C15, C16, C17, C9, JP4, L1, L2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
